Commit message: Driving robot

File: description/robot_core.xacro (robot description, xacro)
@@ -41,4 +41,7 @@
         </xacro:inertial_box>
     </link>
+    <gazebo reference = "chassis">
+        <material>Gazebo/Red</material>
+    </gazebo>
     <!-- LEFT WHEEL LINK -->
     <joint name ="left_wheel_joint" type ="continuous">
@@ -64,4 +67,7 @@
         </xacro:inertial_cylinder>
     </link>
+    <gazebo reference = "left_wheel">
+        <material>Gazebo/Black</material>
+    </gazebo>
         <!-- RIGHT WHEEL LINK -->
         <joint name ="right_wheel_joint" type ="continuous">
@@ -87,4 +93,7 @@
         </xacro:inertial_cylinder>
         </link>
+        <gazebo reference = "right_wheel">
+            <material>Gazebo/Black</material>
+        </gazebo>
         <!-- CASTER WHEEL LINK -->
         <joint name="caster_wheel_joint" type="fixed">
@@ -109,3 +118,6 @@
             </xacro:inertial_sphere>
         </link>
+        <gazebo reference = "caster_wheel">
+            <material>Gazebo/Black</material>
+        </gazebo>
 </robot>

Commit message: mapping

File: description/robot_core.xacro (robot description, xacro)
@@ -16,4 +16,12 @@
     <!-- BASE LINK -->
     <link name ="base_link">
+    </link>
+    <!-- BASE_FOOTPRINT LINK -->
+    <joint name="base_footprint_joint" type="fixed">
+        <parent link="base_link"/>
+        <child link="base_footprint"/>
+        <origin xyz="0 0 0" rpy="0 0 0"/>
+    </joint>
+    <link name="base_footprint">
     </link>
     <!-- CHASSIS LINK -->
