Commit message: Implemented ros2_control

File: description/lidar.xacro (robot description, xacro)
@@ -37,5 +37,5 @@
                 </scan>
                 <range>
-                    <min>0.2</min>
+                    <min>0.18</min>
                     <max>40</max>
                 </range>

File: description/robot.urdf.xacro (robot description, xacro)
@@ -1,6 +1,12 @@
 <?xml version="1.0"?>
 <robot xmlns:xacro="http://www.ros.org/wiki/xacro"  name="robot">
+    <xacro:arg name="use_ros2_control" default="true"/>
     <xacro:include filename="robot_core.xacro" />
-    <xacro:include filename="gazebo_control.xacro" />
+    <xacro:if value="$(arg use_ros2_control)">
+        <xacro:include filename="ros2_control.xacro" />
+    </xacro:if>
+    <xacro:unless value="$(arg use_ros2_control)">
+        <xacro:include filename="gazebo_control.xacro" />
+    </xacro:unless>
     <xacro:include filename="lidar.xacro" />
 </robot>

File: description/robot_core.xacro (robot description, xacro)
@@ -68,5 +68,5 @@
         <collision>
             <geometry>
-                <cylinder radius="0.0325" length="0.027"/>
+                <sphere radius="0.0325"/>
             </geometry>
         </collision>
@@ -94,5 +94,5 @@
             <collision>
                 <geometry>
-                    <cylinder radius="0.0325" length="0.027"/>
+                    <sphere radius="0.0325"/>
                 </geometry>
             </collision>
