Commit message: Implemented teleoperation

File: description/camera.xacro (robot description, xacro)
@@ -4,10 +4,10 @@
         <parent link="chassis"/>
         <child link="camera_link"/>
-        <origin xyz="0.22 0 0.04" rpy="0 0 0"/>
+        <origin xyz="0.2223 0 0.035" rpy="0 0 0"/>
     </joint>
     <link name="camera_link">
         <visual>
             <geometry>
-                <box size="0.010 0.02 0.02"/>
+                <box size="0.005 0.02 0.02"/>
             </geometry>
             <material name="black"/>
@@ -15,5 +15,5 @@
     </link>
     <joint name="camera_joint_optical" type="fixed">
-        <parent link="chassis"/>
+        <parent link="camera_link"/>
         <child link="camera_link_optical"/>
         <origin xyz="0 0 0" rpy="${-pi/2} 0 ${-pi/2}"/>
@@ -25,7 +25,7 @@
             <pose> 0 0 0 0 0 0 </pose>
             <visualize>true</visualize>
-            <update_rate>10</update_rate>
+            <update_rate>31</update_rate>
             <camera>
-                <horizontal_fov>1</horizontal_fov>
+                <horizontal_fov>1.089</horizontal_fov>
                 <image>
                     <width>640</width>

File: description/lidar.xacro (robot description, xacro)
@@ -26,5 +26,5 @@
         <sensor name="laser" type="ray">
             <pose> 0 0 0 0 0 0 </pose>
-            <visualize>false</visualize>
+            <visualize>false</visualize> <!-- Set to true to visualize the rays -->
             <update_rate>10</update_rate>
             <ray>

File: description/robot_core.xacro (robot description, xacro)
@@ -45,5 +45,5 @@
             </geometry>
         </collision>
-        <xacro:inertial_box mass="0.5" x="0.22" y="0.14" z="0.07">
+        <xacro:inertial_box mass="0.8" x="0.22" y="0.14" z="0.07">
             <origin xyz="0.11 0 0.035" rpy="0 0 0"/>
         </xacro:inertial_box>

Commit message: Update configuration files for simulation environment and for the real robot

File: description/camera.xacro (robot description, xacro)
@@ -4,5 +4,5 @@
         <parent link="chassis"/>
         <child link="camera_link"/>
-        <origin xyz="0.2223 0 0.035" rpy="0 0 0"/>
+        <origin xyz="0.3323 0 0.1" rpy="0 0 0"/>
     </joint>
     <link name="camera_link">
@@ -25,5 +25,5 @@
             <pose> 0 0 0 0 0 0 </pose>
             <visualize>true</visualize>
-            <update_rate>31</update_rate>
+            <update_rate>10</update_rate>
             <camera>
                 <horizontal_fov>1.089</horizontal_fov>

File: description/gazebo_control.xacro (robot description, xacro)
@@ -6,6 +6,6 @@
              <left_joint>left_wheel_joint</left_joint>
              <right_joint>right_wheel_joint</right_joint>
-             <wheel_separation>0.172</wheel_separation>
-             <wheel_diameter>0.065</wheel_diameter>
+             <wheel_separation>0.2116</wheel_separation>
+             <wheel_diameter>0.069</wheel_diameter>
             <!-- Limits-->
              <max_wheel_torque>200</max_wheel_torque>

File: description/lidar.xacro (robot description, xacro)
@@ -4,5 +4,5 @@
         <parent link="chassis"/>
         <child link="lidar_frame"/>
-        <origin xyz="0.15 0 0.08" rpy="0 0 0"/>
+        <origin xyz="0.165 0 0.16" rpy="0 0 0"/>
     </joint>
     <link name="lidar_frame">

File: description/robot.urdf.xacro (robot description, xacro)
@@ -2,4 +2,5 @@
 <robot xmlns:xacro="http://www.ros.org/wiki/xacro"  name="robot">
     <xacro:arg name="use_ros2_control" default="true"/>
+    <xacro:arg name="sim_mode" default="false"/>
     <xacro:include filename="robot_core.xacro" />
     <xacro:if value="$(arg use_ros2_control)">

File: description/robot_core.xacro (robot description, xacro)
@@ -29,22 +29,22 @@
         <parent link="base_link"/>
         <child link="chassis"/>
-        <origin xyz="-0.073333333 0 0"/>
+        <origin xyz="-0.065 0 0"/>
     </joint>
     <link name="chassis">
         <visual>
-            <origin xyz="0.11 0 0.035"/>
+            <origin xyz="0.165 0 0.075"/>
             <geometry>
-                <box size="0.22 0.14 0.07"/>
+                <box size="0.33 0.19 0.15"/>
             </geometry>
             <material name="red"/>
         </visual>
         <collision>
-            <origin xyz="0.11 0 0.035"/>
+            <origin xyz="0.165 0 0.075"/>
             <geometry>
-                <box size="0.22 0.14 0.07"/>
+                <box size="0.33 0.19 0.15"/>
             </geometry>
         </collision>
-        <xacro:inertial_box mass="0.8" x="0.22" y="0.14" z="0.07">
-            <origin xyz="0.11 0 0.035" rpy="0 0 0"/>
+        <xacro:inertial_box mass="0.8" x="0.33" y="0.19" z="0.15">
+            <origin xyz="0.165 0 0.075" rpy="0 0 0"/>
         </xacro:inertial_box>
     </link>
@@ -56,5 +56,5 @@
         <parent link = "base_link"/>
         <child link = "left_wheel"/>
-        <origin xyz="0 0.086 0" rpy="-${pi/2} 0 0"/>
+        <origin xyz="0 0.1084 0" rpy="-${pi/2} 0 0"/>
         <axis xyz="0 0 1"/>
     </joint>
@@ -71,5 +71,5 @@
             </geometry>
         </collision>
-        <xacro:inertial_cylinder mass="0.08" length="0.027" radius="0.0325">
+        <xacro:inertial_cylinder mass="0.2" length="0.027" radius="0.0325">
             <origin xyz="0 0 0" rpy="0 0 0"/>
         </xacro:inertial_cylinder>
@@ -82,5 +82,5 @@
             <parent link = "base_link"/>
             <child link = "right_wheel"/>
-            <origin xyz="0 -0.086 0" rpy="${pi/2} 0 0"/>
+            <origin xyz="0 -0.1084 0" rpy="${pi/2} 0 0"/>
             <axis xyz="0 0 -1"/>
         </joint>
@@ -97,5 +97,5 @@
                 </geometry>
             </collision>
-            <xacro:inertial_cylinder mass="0.08" length="0.027" radius="0.0325">
+            <xacro:inertial_cylinder mass="0.2" length="0.027" radius="0.0325">
             <origin xyz="0 0 0" rpy="0 0 0"/>
         </xacro:inertial_cylinder>
@@ -108,5 +108,5 @@
             <parent link="chassis"/>
             <child link="caster_wheel"/>
-            <origin xyz="0.18 0 0"/>
+            <origin xyz="0.27 0 0"/>
         </joint>
         <link name="caster_wheel">
@@ -122,5 +122,5 @@
                 </geometry>
             </collision>
-            <xacro:inertial_sphere mass="0.2" radius="0.0325">
+            <xacro:inertial_sphere mass="0.3" radius="0.0325">
                 <origin xyz="0 0 0" rpy="0 0 0"/>
             </xacro:inertial_sphere>
@@ -128,6 +128,6 @@
         <gazebo reference = "caster_wheel">
             <material>Gazebo/Black</material>
-            <mu1 value="0.001"/>
-            <mu2 value="0.001"/>
+            <mu1 value="0.005"/>
+            <mu2 value="0.005"/>
         </gazebo>
 </robot>

File: description/ros2_control.xacro (robot description, xacro)
@@ -1,30 +1,62 @@
 <?xml version="1.0"?>
 <robot xmlns:xacro="http://www.ros.org/wiki/xacro">
-  <ros2_control name="GazeboSimSystem" type="system">
-    <hardware>
-      <plugin>gazebo_ros2_control/GazeboSystem</plugin>
-    </hardware>
-    <joint name="left_wheel_joint">
-      <command_interface name="velocity">
-        <param name="min">-10</param>
-        <param name="max">10</param>
-      </command_interface>
-      <state_interface name="velocity"/>
-      <state_interface name="position"/>
-    </joint>
-    <joint name="right_wheel_joint">
-      <command_interface name="velocity">
-        <param name="min">-10</param>
-        <param name="max">10</param>
-      </command_interface>
-      <state_interface name="velocity"/>
-      <state_interface name="position"/>
-    </joint>
-  </ros2_control>
-  <gazebo>
-    <plugin name="ros2_control_gazebo" filename="libgazebo_ros2_control.so">
-      <robotNamespace>/my_robot</robotNamespace>
-      <parameters>$(find robot_mobil)/config/controllers.yaml</parameters>
-    </plugin>
-  </gazebo>
+    <xacro:unless value="$(arg sim_mode)">
+        <ros2_control name="RealRobot" type="system">
+            <hardware>
+                <plugin>diffdrive_arduino/DiffDriveArduino</plugin>
+                <param name="left_wheel_name">left_wheel_joint</param>
+                <param name="right_wheel_name">right_wheel_joint</param>
+                <param name="loop_rate">30</param>
+                <param name="device">/dev/ttyUSB0</param>
+                <param name="baud_rate">57600</param>
+                <param name="timeout">1000</param>
+                <param name="enc_counts_per_rev">180</param>
+            </hardware>
+            <joint name="left_wheel_joint">
+                <command_interface name="velocity">
+                    <param name="min">-10</param>
+                    <param name="max">10</param>
+                </command_interface>
+                <state_interface name="velocity"/>
+                <state_interface name="position"/>
+            </joint>
+            <joint name="right_wheel_joint">
+                <command_interface name="velocity">
+                    <param name="min">-10</param>
+                    <param name="max">10</param>
+                </command_interface>
+                <state_interface name="velocity"/>
+                <state_interface name="position"/>
+            </joint>
+        </ros2_control>
+    </xacro:unless>
+    <xacro:if value="$(arg sim_mode)">
+        <ros2_control name="GazeboSystem" type="system">
+            <hardware>
+                <plugin>gazebo_ros2_control/GazeboSystem</plugin>
+            </hardware>
+            <joint name="left_wheel_joint">
+                <command_interface name="velocity">
+                    <param name="min">-10</param>
+                    <param name="max">10</param>
+                </command_interface>
+                <state_interface name="velocity"/>
+                <state_interface name="position"/>
+            </joint>
+            <joint name="right_wheel_joint">
+                <command_interface name="velocity">
+                    <param name="min">-10</param>
+                    <param name="max">10</param>
+                </command_interface>
+                <state_interface name="velocity"/>
+                <state_interface name="position"/>
+            </joint>
+        </ros2_control>
+    </xacro:if>
+    <gazebo>
+        <plugin name="gazebo_ros2_control" filename="libgazebo_ros2_control.so">
+            <parameters>$(find robot_mobil)/config/my_controllers.yaml</parameters>
+            <parameters>$(find robot_mobil)/config/gaz_ros2_ctl_use_sim.yaml</parameters>
+        </plugin>
+    </gazebo>
 </robot>
