Commit message: Added lidar

File: description/gazebo_control.xacro (robot description, xacro)
@@ -6,5 +6,5 @@
              <left_joint>left_wheel_joint</left_joint>
              <right_joint>right_wheel_joint</right_joint>
-             <wheel_separation>0.235</wheel_separation>
+             <wheel_separation>0.172</wheel_separation>
              <wheel_diameter>0.065</wheel_diameter>
             <!-- Limits-->

File: description/robot_core.xacro (robot description, xacro)
@@ -21,25 +21,25 @@
         <parent link="base_link"/>
         <child link="chassis"/>
-        <origin xyz="-0.1 0 0"/>
+        <origin xyz="-0.073333333 0 0"/>
     </joint>
     <link name="chassis">
         <visual>
-            <origin xyz="0.1 0 0.05"/>
+            <origin xyz="0.11 0 0.035"/>
             <geometry>
-                <box size="0.2 0.2 0.1"/>
+                <box size="0.22 0.14 0.07"/>
             </geometry>
             <material name="red"/>
         </visual>
         <collision>
-            <origin xyz="0.1 0 0.05"/>
+            <origin xyz="0.11 0 0.035"/>
             <geometry>
-                <box size="0.2 0.2 0.1"/>
+                <box size="0.22 0.14 0.07"/>
             </geometry>
         </collision>
-        <xacro:inertial_box mass="0.4" x="0.2" y="0.2" z="0.1">
-            <origin xyz="0.1 0 0.05" rpy="0 0 0"/>
+        <xacro:inertial_box mass="0.5" x="0.22" y="0.14" z="0.07">
+            <origin xyz="0.11 0 0.035" rpy="0 0 0"/>
         </xacro:inertial_box>
     </link>
-    <gazebo reference = "chassis">
+    <gazebo reference="chassis">
         <material>Gazebo/Red</material>
     </gazebo>
@@ -48,5 +48,5 @@
         <parent link = "base_link"/>
         <child link = "left_wheel"/>
-        <origin xyz="-0.030 0.1175 0" rpy="-${pi/2} 0 0"/>
+        <origin xyz="0 0.086 0" rpy="-${pi/2} 0 0"/>
         <axis xyz="0 0 1"/>
     </joint>
@@ -54,5 +54,5 @@
         <visual>
             <geometry>
-                <cylinder radius="0.04" length="0.03"/>
+                <cylinder radius="0.0325" length="0.027"/>
             </geometry>
             <material name="black"/>
@@ -60,8 +60,8 @@
         <collision>
             <geometry>
-                <cylinder radius="0.04" length="0.03"/>
+                <cylinder radius="0.0325" length="0.027"/>
             </geometry>
         </collision>
-        <xacro:inertial_cylinder mass="0.08" length="0.03" radius="0.04">
+        <xacro:inertial_cylinder mass="0.08" length="0.027" radius="0.0325">
             <origin xyz="0 0 0" rpy="0 0 0"/>
         </xacro:inertial_cylinder>
@@ -74,5 +74,5 @@
             <parent link = "base_link"/>
             <child link = "right_wheel"/>
-            <origin xyz="-0.030 -0.1175 0" rpy="${pi/2} 0 0"/>
+            <origin xyz="0 -0.086 0" rpy="${pi/2} 0 0"/>
             <axis xyz="0 0 -1"/>
         </joint>
@@ -80,5 +80,5 @@
             <visual>
                 <geometry>
-                    <cylinder radius="0.04" length="0.03"/>
+                    <cylinder radius="0.0325" length="0.027"/>
                 </geometry>
                 <material name="black"/>
@@ -86,8 +86,8 @@
             <collision>
                 <geometry>
-                    <cylinder radius="0.04" length="0.03"/>
+                    <cylinder radius="0.0325" length="0.027"/>
                 </geometry>
             </collision>
-            <xacro:inertial_cylinder mass="0.08" length="0.03" radius="0.04">
+            <xacro:inertial_cylinder mass="0.08" length="0.027" radius="0.0325">
             <origin xyz="0 0 0" rpy="0 0 0"/>
         </xacro:inertial_cylinder>
@@ -100,10 +100,10 @@
             <parent link="chassis"/>
             <child link="caster_wheel"/>
-            <origin xyz="0.16 0 0"/>
+            <origin xyz="0.18 0 0"/>
         </joint>
         <link name="caster_wheel">
             <visual>
                 <geometry>
-                    <sphere radius="0.04"/>
+                    <sphere radius="0.0325"/>
                 </geometry>
                 <material name="black"/>
@@ -111,8 +111,8 @@
             <collision>
                 <geometry>
-                    <sphere radius="0.04"/>
+                    <sphere radius="0.0325"/>
                 </geometry>
             </collision>
-            <xacro:inertial_sphere mass="0.15" radius="0.04">
+            <xacro:inertial_sphere mass="0.2" radius="0.0325">
                 <origin xyz="0 0 0" rpy="0 0 0"/>
             </xacro:inertial_sphere>

Commit message: Implemented autonomous navigation and object tracking

File: description/gazebo_control.xacro (robot description, xacro)
@@ -6,5 +6,5 @@
              <left_joint>left_wheel_joint</left_joint>
              <right_joint>right_wheel_joint</right_joint>
-             <wheel_separation>0.2116</wheel_separation>
+             <wheel_separation>0.22</wheel_separation>
              <wheel_diameter>0.069</wheel_diameter>
             <!-- Limits-->

File: description/robot_core.xacro (robot description, xacro)
@@ -56,5 +56,5 @@
         <parent link = "base_link"/>
         <child link = "left_wheel"/>
-        <origin xyz="0 0.1084 0" rpy="-${pi/2} 0 0"/>
+        <origin xyz="0 0.11 0" rpy="-${pi/2} 0 0"/>
         <axis xyz="0 0 1"/>
     </joint>
@@ -82,5 +82,5 @@
             <parent link = "base_link"/>
             <child link = "right_wheel"/>
-            <origin xyz="0 -0.1084 0" rpy="${pi/2} 0 0"/>
+            <origin xyz="0 -0.11 0" rpy="${pi/2} 0 0"/>
             <axis xyz="0 0 -1"/>
         </joint>

File: description/ros2_control.xacro (robot description, xacro)
@@ -11,5 +11,5 @@
                 <param name="baud_rate">57600</param>
                 <param name="timeout">1000</param>
-                <param name="enc_counts_per_rev">180</param>
+                <param name="enc_counts_per_rev">7248</param>
             </hardware>
             <joint name="left_wheel_joint">
